Commit message: fixed_urdf

File: urdf/ur_macro.xacro (robot description, xacro)
@@ -315,16 +315,13 @@
       </inertial>
     </link>
-    <!-- link name="endeffector_type5" -->
-    <link name="endeffector_type6" >
-      <visual>
-        <geometry>
-          <!-- mesh filename="package://harvesting_endeffector/type5/ee_type5.stl"/ -->
-          <mesh filename="package://harvesting_endeffector/type6/linear_cutting_endeffector-short_mirrer-main.stl" scale="0.001 0.001 0.001"/>
-        </geometry>
-      </visual>
-      <collision>
-        <geometry>
-          <!-- mesh filename="package://harvesting_endeffector/type5/ee_type5.stl"/ -->
-          <mesh filename="package://harvesting_endeffector/type6/linear_cutting_endeffector-short_mirrer-main.stl" scale="0 0 0"/>
+    <link name="endeffector_type5">
+      <visual>
+        <geometry>
+          <mesh filename="package://harvesting_endeffector/type5/ee_type5.stl"/>
+        </geometry>
+      </visual>
+      <collision>
+        <geometry>
+          <mesh filename="package://harvesting_endeffector/type5/ee_type5.stl"/>
         </geometry>
       </collision>
@@ -334,4 +331,20 @@
       </inertial>
     </link>
+    <!-- <link name="endeffector_type6" >
+      <visual>
+        <geometry>
+          <mesh filename="package://harvesting_endeffector/type6/linear_cutting_endeffector-short_mirrer-main.stl" scale="0.001 0.001 0.001"/>
+        </geometry>
+      </visual>
+      <collision>
+        <geometry>
+          <mesh filename="package://harvesting_endeffector/type6/linear_cutting_endeffector-short_mirrer-main.stl" scale="0.001 0.001 0.001"/>
+        </geometry>
+      </collision>
+      <inertial>
+        <mass value="0.1"/>
+        <inertia ixx="0.00042" iyy="0.00042" izz="0.00042" ixy="0" ixz="0" iyz="0" />
+      </inertial>
+    </link> -->
     <link name="endeffector_base">
       <visual>
@@ -573,14 +586,16 @@
       <origin xyz="0 0 0.05" rpy="-${pi/2.0} -${pi/2.0} 0"/>
       <parent link="endeffector_base"/>
-      <!-- child link="endeffector_type5"/ -->
+      <child link="endeffector_type5"/>
+    </joint>
+    <!-- <joint name="eebase_to_ee" type="fixed">
+      <origin xyz="0 0 0.105" rpy="-${pi/2.0} -${pi/2.0} 0"/>
+      <parent link="endeffector_base"/>
       <child link="endeffector_type6"/>
-    </joint>
+    </joint> -->
     <joint name="ee_to_cutter" type="fixed">
-      <!-- origin xyz="0.315 -0.01 -0.024" rpy="${pi/2.0} 0 ${pi/2.0}"/ -->
-      <origin xyz="0.18 0.0 0.0" rpy="${pi/2.0} 0 ${pi/2.0}"/>
-      <!-- -0.028 -->
-      <!-- 0.025 -->
-      <!-- parent link="endeffector_type5"/ -->
-      <parent link="endeffector_type6"/>
+      <origin xyz="0.315 -0.01 -0.024" rpy="${pi/2.0} 0 ${pi/2.0}"/>
+      <!-- <origin xyz="0.18 -0.01 -0.005" rpy="${pi/2.0} 0 ${pi/2.0}"/> -->
+      <!-- <parent link="endeffector_type5"/> -->
+      <parent link="endeffector_type5"/>
       <child link="endeffector_cutter"/>
     </joint>

Commit message: fixed_path

File: urdf/ur_macro.xacro (robot description, xacro)
@@ -315,5 +315,5 @@
       </inertial>
     </link>
-    <link name="endeffector_type5">
+    <!-- <link name="endeffector_type5">
       <visual>
         <geometry>
@@ -330,6 +330,6 @@
         <inertia ixx="0.00042" iyy="0.00042" izz="0.00042" ixy="0" ixz="0" iyz="0" />
       </inertial>
-    </link>
-    <!-- <link name="endeffector_type6" >
+    </link> -->
+    <link name="endeffector_type6" >
       <visual>
         <geometry>
@@ -346,5 +346,5 @@
         <inertia ixx="0.00042" iyy="0.00042" izz="0.00042" ixy="0" ixz="0" iyz="0" />
       </inertial>
-    </link> -->
+    </link>
     <link name="endeffector_base">
       <visual>
@@ -583,19 +583,22 @@
       <child link="realsense_cable"/>
     </joint>
-    <joint name="eebase_to_ee" type="fixed">
+    <!-- <joint name="eebase_to_ee" type="fixed">
       <origin xyz="0 0 0.05" rpy="-${pi/2.0} -${pi/2.0} 0"/>
       <parent link="endeffector_base"/>
       <child link="endeffector_type5"/>
     </joint>
-    <!-- <joint name="eebase_to_ee" type="fixed">
+    <joint name="ee_to_cutter" type="fixed">
+      <origin xyz="0.315 -0.01 -0.024" rpy="${pi/2.0} 0 ${pi/2.0}"/>
+      <parent link="endeffector_type5"/>
+      <child link="endeffector_cutter"/>
+    </joint> -->
+    <joint name="eebase_to_ee" type="fixed">
       <origin xyz="0 0 0.105" rpy="-${pi/2.0} -${pi/2.0} 0"/>
       <parent link="endeffector_base"/>
       <child link="endeffector_type6"/>
-    </joint> -->
+    </joint>
     <joint name="ee_to_cutter" type="fixed">
-      <origin xyz="0.315 -0.01 -0.024" rpy="${pi/2.0} 0 ${pi/2.0}"/>
-      <!-- <origin xyz="0.18 -0.01 -0.005" rpy="${pi/2.0} 0 ${pi/2.0}"/> -->
-      <!-- <parent link="endeffector_type5"/> -->
-      <parent link="endeffector_type5"/>
+      <origin xyz="0.18 -0.01 -0.005" rpy="${pi/2.0} 0 ${pi/2.0}"/>
+      <parent link="endeffector_type6"/>
       <child link="endeffector_cutter"/>
     </joint>

Commit message: add_vertical_base

File: urdf/ur_macro.xacro (robot description, xacro)
@@ -339,5 +339,5 @@
           <!-- mesh filename="package://harvesting_endeffector/type5/ee_base.stl"/ -->
           <!--mesh filename="package://harvesting_endeffector/type6/Final.stl" scale="0.001 0.001 0.001"/ -->
-          <mesh filename="package://harvesting_endeffector/type6/EndEffector_inventor_2024smailscale.stl"/>
+          <mesh filename="package://harvesting_endeffector/type7/EndEffector_Verical_v2.stl" scale="0.001 0.001 0.001"/>
         </geometry>
       </visual>
@@ -346,5 +346,5 @@
           <!-- mesh filename="package://harvesting_endeffector/type5/ee_base.stl"/ -->
           <!-- mesh filename="package://harvesting_endeffector/type6/Final.stl" scale="0.001 0.001 0.001"/ -->
-          <mesh filename="package://harvesting_endeffector/type6/EndEffector_inventor_2024smailscale.stl"/>
+          <mesh filename="package://harvesting_endeffector/type7/EndEffector_Verical_v2.stl" scale="0.001 0.001 0.001"/>
         </geometry>
       </collision>
@@ -556,10 +556,10 @@
     </joint>
     <joint name="tool0_to_ee_base" type="fixed">
-      <origin xyz="0 0 0.001" rpy="0.0 0.0 ${pi}"/>
+      <origin xyz="0 0 -0.05" rpy="0.0 0.0 0.0"/>
       <parent link="${tf_prefix}tool0"/>
       <child link="endeffector_base"/>
     </joint>
     <xacro:sensor_d435 parent="endeffector_base" name="head_camera">
-      <origin xyz="0 0.080 0.014" rpy="-1.5708 -1.5708 0"/>
+      <origin xyz="0 0.080 0.014" rpy="0 0 ${pi/2.0}"/>
       <!-- origin xyz="0 0.074 0.06" rpy="0.0 -1.5271630953540196 -1.570876783818119"/ -->
       <!-- <origin xyz="0 0.074 0.06" rpy="-1.570834 -1.483529 3.14155050"/> -->
@@ -575,5 +575,5 @@
     </joint>
     <joint name="eebase_to_ee" type="fixed">
-      <origin xyz="0.01 0.0025 0.101" rpy="-${pi/2.0} -${pi/2.0} 0"/>
+      <origin xyz="-0.01 0.167 0.0966" rpy="0 0 ${pi/2.0}"/>
       <parent link="endeffector_base"/>
       <!-- child link="endeffector_type5"/ -->
@@ -582,5 +582,5 @@
     <joint name="ee_to_cutter" type="fixed">
       <!-- origin xyz="0.315 -0.01 -0.024" rpy="${pi/2.0} 0 ${pi/2.0}"/ -->
-      <origin xyz="0.18 -0.01 -0.005" rpy="${pi/2.0} 0 ${pi/2.0}"/>
+      <origin xyz="0.18 -0.01 -0.01" rpy="${pi/2.0} 0 ${pi/2.0}"/>
       <!-- -0.028 -->
       <!-- 0.025 -->

Commit message: 関節制限変更，手先の姿勢変更

File: urdf/ur_macro.xacro (robot description, xacro)
@@ -339,5 +339,5 @@
           <!-- mesh filename="package://harvesting_endeffector/type5/ee_base.stl"/ -->
           <!--mesh filename="package://harvesting_endeffector/type6/Final.stl" scale="0.001 0.001 0.001"/ -->
-          <mesh filename="package://harvesting_endeffector/type7/EndEffector_Verical_v2.stl" scale="0.001 0.001 0.001"/>
+          <mesh filename="package://harvesting_endeffector/type7/EndEffector_Verical_v2_double.stl"/>
         </geometry>
       </visual>
@@ -346,5 +346,5 @@
           <!-- mesh filename="package://harvesting_endeffector/type5/ee_base.stl"/ -->
           <!-- mesh filename="package://harvesting_endeffector/type6/Final.stl" scale="0.001 0.001 0.001"/ -->
-          <mesh filename="package://harvesting_endeffector/type7/EndEffector_Verical_v2.stl" scale="0.001 0.001 0.001"/>
+          <mesh filename="package://harvesting_endeffector/type7/EndEffector_Verical_v2_double.stl"/>
         </geometry>
       </collision>
@@ -555,6 +555,11 @@
       <child link="${tf_prefix}tool0"/>
     </joint>
+    <!-- <joint name="tool0_to_ee_base" type="fixed">
+      <origin xyz="0 0 -0.05" rpy="0.0 0.0 0.0"/>
+      <parent link="${tf_prefix}tool0"/>
+      <child link="endeffector_base"/>
+    </joint> -->
     <joint name="tool0_to_ee_base" type="fixed">
-      <origin xyz="0 0 -0.05" rpy="0.0 0.0 0.0"/>
+      <origin xyz="0 0 0.138" rpy="0.0 ${pi} 0.0"/>
       <parent link="${tf_prefix}tool0"/>
       <child link="endeffector_base"/>

Commit message: change param

File: urdf/ur_macro.xacro (robot description, xacro)
@@ -422,10 +422,10 @@
     </joint>
     <joint name="base_link_to_cart_collider" type="fixed">
-      <origin xyz="-0.25 0 -0.151" rpy="0 0 0"/>
+      <origin xyz="-0.3 0 -0.151" rpy="0 0 0"/>
       <parent link="${tf_prefix}base_link"/>
       <child link="cart_collider"/>
     </joint>
     <joint name="base_link_to_arm_collider" type="fixed">
-      <origin xyz="-0.4 0 0.251" rpy="0 0 0"/>
+      <origin xyz="-0.55 0 0.251" rpy="0 0 0"/>
       <parent link="${tf_prefix}base_link"/>
       <child link="arm_collider"/>
@@ -566,5 +566,5 @@
     </joint>
     <xacro:sensor_d435 parent="endeffector_base" name="head_camera">
-      <origin xyz="0 0.080 0.014" rpy="0 0 ${pi/2.0}"/>
+      <origin xyz="0 0.080 -0.011" rpy="0 0 ${pi/2.0}"/>
       <!-- origin xyz="0 0.074 0.06" rpy="0.0 -1.5271630953540196 -1.570876783818119"/ -->
       <!-- <origin xyz="0 0.074 0.06" rpy="-1.570834 -1.483529 3.14155050"/> -->
